File: usdex_card-to-fpc/usdex_card-to-fpc.kicad_pcb (KiCad board)
At the start: 6 copper layers, 11 x 15 mm, 2 parts, among them J1 Micro_SDex_PCB, J2 Conn_01x16_Socket

Commit message: WIP
Parts:
- J2: footprint m1cha:1x16_FPC_solder -> m1cha:usdex-fpc-1x16-0.64mm
- moved J2 0.43 mm to (-0.65, 16.2)
Connections:
- net REFCLK+/DAT0 renamed DATx/REFCLK+
- net REFCLK-/DAT1 renamed DATx/REFCLK-
Routing:
- net CMD: track 15.3 -> 0.00 mm, vias 1 -> 0
- net GND: track 0.00 -> 14.3 mm, vias 1 -> 5
- net +1V8: track 0.00 -> 12.9 mm, vias 0 -> 1
- net +3V3: track 0.00 -> 2.33 mm, vias 1 -> 2
- net CLK: track 15.6 -> 15.1 mm

Commit message: finish usdex card
Parts:
- J2: footprint m1cha:usdex-fpc-1x16-0.64mm -> m1cha:usdex-fpc-1x18-0.55mm
Routing:
- net GND: track 14.3 -> 31.0 mm, vias 5 -> 14
- net CMD: track 0.00 -> 14.7 mm, vias 0 -> 1
- net +3V3: track 2.33 -> 3.53 mm, vias 2 -> 5
- net +1V8: track 12.9 -> 12.1 mm
- net ~{CLKREQ}/DAT2: track 14.9 -> 14.3 mm
- net ~{PERST}/DAT3/CD: track 15.0 -> 14.5 mm
