File: usdex_card-to-fpc/usdex_card-to-fpc.kicad_sch (KiCad schematic)
At the start: 2 parts, among them J1 Micro_SDex_PCB, J2 Conn_01x16_Socket

Commit message: WIP
Parts:
- J2: footprint m1cha:1x16_FPC_solder -> m1cha:usdex-fpc-1x16-0.64mm
Connections:
- net REFCLK+/DAT0 renamed DATx/REFCLK+
- net REFCLK-/DAT1 renamed DATx/REFCLK-
Changed lines of the file:
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@@
 		)
 	)
-	(global_label "REFCLK-{slash}DAT1"
+	(global_label "DATx{slash}REFCLK-"
 		(shape input)
 		(at 45.72 100.33 180)
@@
 		)
 		(property "Intersheetrefs" "${INTERSHEET_REFS}"
-			(at 28.2205 100.33 0)
-			(effects
-				(font
-					(size 1.27 1.27)
-				)
-				(justify right)
-				(hide yes)
-			)
-		)
-	)
-	(global_label "REFCLK-{slash}DAT1"
+			(at 28.4019 100.33 0)
+			(effects
+				(font
+					(size 1.27 1.27)
+				)
+				(justify right)
+				(hide yes)
+			)
+		)
+	)
+	(global_label "DATx{slash}REFCLK-"
 		(shape input)
 		(at 36.83 38.1 180)
@@
 		)
 		(property "Intersheetrefs" "${INTERSHEET_REFS}"
-			(at 19.3305 38.1 0)
+			(at 19.5119 38.1 0)
 			(effects
 				(font
@@
 		)
 	)
-	(global_label "REFCLK+{slash}DAT0"
+	(global_label "DATx{slash}REFCLK+"
 		(shape input)
 		(at 36.83 35.56 180)
@@
 		)
 		(property "Intersheetrefs" "${INTERSHEET_REFS}"
-			(at 19.3305 35.56 0)
+			(at 19.5119 35.56 0)
 			(effects
 				(font
@@
 		)
 	)
-	(global_label "REFCLK+{slash}DAT0"
+	(global_label "DATx{slash}REFCLK+"
 		(shape input)
 		(at 45.72 102.87 180)
@@
 		)
 		(property "Intersheetrefs" "${INTERSHEET_REFS}"
-			(at 28.2205 102.87 0)
+			(at 28.4019 102.87 0)
 			(effects
 				(font
@@
 			)
 		)
-		(property "Footprint" "m1cha:1x16_FPC_solder"
+		(property "Footprint" "m1cha:usdex-fpc-1x16-0.64mm"
 			(at 50.8 97.79 0)
 			(effects

Commit message: finish usdex card
Parts:
- J2: footprint m1cha:usdex-fpc-1x16-0.64mm -> m1cha:usdex-fpc-1x18-0.55mm
Other:
- moved on the sheet: J2
