File: fpc-to-m2_m_socket/fpc-to-m2_m_socket.kicad_pcb (KiCad board)
At the start: 6 copper layers, 100 x 43.5 mm, 21 parts, among them J2 Bus_M.2_Socket_M, Y1 OK2EL89CJI-111YLC-32.768K

Commit message: that should work
Parts:
- moved R2 12.2 mm to (128.9, 88.6)
- moved R3 12.2 mm to (127.8, 88.6)
- moved C1 7.25 mm to (123.0, 71.6), turned to 180 degrees
- moved U2 4.31 mm to (121.7, 75.0)
- moved R4 1.98 mm to (86.0, 105.6)
- moved C4 1.54 mm to (84.7, 106.1)
- moved C2 0.96 mm to (98.1, 82.4)
- moved C3 0.96 mm to (97.1, 82.4)
Routing:
- net ~{LED1}: track 0.00 -> 47.7 mm
- net Net-(J2-VIO_1.8V): track 0.00 -> 37.2 mm
- net Net-(J2-DEVSLP): track 0.00 -> 34.5 mm
- net CMD: track 0.00 -> 34.5 mm, vias 0 -> 1
- net CLK: track 0.00 -> 31.5 mm, vias 0 -> 1
- net DAT0: track 0.00 -> 29.4 mm, vias 0 -> 1
- net DAT1: track 0.00 -> 29.2 mm, vias 0 -> 1
- net SUSCLK: track 0.00 -> 21.5 mm, vias 0 -> 2
- net ~{CLKREQ}: track 32.4 -> 48.8 mm
- net ~{PERST}: track 29.4 -> 40.6 mm, vias 0 -> 2
- net DAT3/CD: track 0.00 -> 5.15 mm, vias 0 -> 1
- net DAT2: track 0.00 -> 4.54 mm, vias 0 -> 1
- net ~{CLKREQ}/DAT2: track 28.6 -> 31.6 mm, vias 0 -> 2
- net PCIe_TX-: track 29.5 -> 31.9 mm, vias 0 -> 2
- net Net-(D1-K): track 0.00 -> 2.29 mm
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
Commit message: reduce width
Parts:
- moved C3 7.23 mm to (89.9, 82.4)
- moved R1 7.23 mm to (96.0, 82.2)
- moved U1 7.23 mm to (93.6, 82.2)
- moved C2 7.23 mm to (90.8, 82.4)
- moved J1 7.20 mm to (94.6, 78.1)
Routing:
- net CMD: track 34.5 -> 0.00 mm, vias 1 -> 0
- net ~{CLKREQ}/DAT2: track 31.6 -> 0.00 mm, vias 2 -> 0
- net CLK: track 31.5 -> 0.00 mm, vias 1 -> 0
- net ~{PERST}/DAT3/CD: track 30.2 -> 0.00 mm, vias 2 -> 0
- net DAT0: track 29.4 -> 0.00 mm, vias 1 -> 0
- net DAT1: track 29.2 -> 0.00 mm, vias 1 -> 0
- net PCIe_RX+: track 40.7 -> 34.6 mm
- net PCIe_RX-: track 41.5 -> 35.3 mm
- net PCIe_TX+: track 30.9 -> 33.7 mm
- net PCIe_TX-: track 31.9 -> 34.4 mm
- net REFCLK-: track 19.4 -> 17.9 mm
- net REFCLK+: track 18.7 -> 17.1 mm
Other:
- board size 100 x 43.5 mm -> 98.3 x 43.5 mm

Commit message: WIP
Parts:
- moved C5 11.8 mm to (162.0, 88.0)
- moved C1 3.49 mm to (123.0, 75.0)
- moved U2 3.49 mm to (121.7, 78.5)
- moved C3 3.37 mm to (91.7, 85.2)
- moved J3 3.30 mm to (150.0, 76.5)
- moved J4 3.25 mm to (171.0, 81.5)
- moved J1 3.01 mm to (95.2, 81.1)
- moved U1 3.01 mm to (94.1, 85.2)
- moved R1 3.00 mm to (96.5, 85.1)
- moved C2 2.81 mm to (90.8, 85.2)
Routing:
- net ~{CLKREQ}: track 48.8 -> 39.0 mm
- net ~{PERST}: track 40.6 -> 32.1 mm
- net REFCLK-: track 17.9 -> 15.1 mm
- net REFCLK+: track 17.1 -> 14.4 mm
- net PCIe_RX-: track 35.3 -> 32.7 mm
- net PCIe_RX+: track 34.6 -> 32.1 mm
- net PCIe_TX-: track 34.4 -> 32.6 mm
- net PCIe_TX+: track 33.7 -> 31.9 mm
Other:
- board size 98.3 x 43.5 mm -> 98.3 x 40.6 mm

Commit message: almost done
Parts:
- added J5: Conn_01x02_Pin, Connector_PinHeader_2.54mm:PinHeader_1x02_P2.54mm_Vertical, F.Cu at (83.5, 89.2)
- J1: footprint m1cha:FPC-SMD_P1.00-16P_LCS-SJ-H2.5 -> m1cha:FPC-SMD_18P-P1.00_JS_AFA07-S18XXX
- Y1: footprint Oscillator:Oscillator_SMD_Abracon_ASDMB-4Pin_2.5x2.0mm -> m1cha:OSC-SMD_4P-L3.2-W2.5-BL_TG-5006CE
- moved R3 18.9 mm to (109.0, 89.2), turned to 180 degrees
- moved R2 17.6 mm to (111.3, 88.6)
- moved R1 12.8 mm to (109.0, 88.1), turned to 0 degrees
- moved D1 11.2 mm to (153.2, 88.0)
- moved R7 11.2 mm to (149.5, 88.0)
- moved C1 4.67 mm to (125.3, 79.1), turned to -90 degrees
- moved C6 3.58 mm to (87.3, 105.0), turned to 90 degrees
- moved R5 1.92 mm to (82.8, 108.1)
- moved C4 1.76 mm to (83.0, 105.5), turned to 180 degrees
- moved R4 1.45 mm to (84.7, 105.0)
- moved R6 1.42 mm to (86.0, 111.2)
- moved C3 0.99 mm to (90.8, 85.3)
- moved C2 0.99 mm to (89.8, 85.3)
- moved J1 0.95 mm to (94.2, 81.1), turned to 180 degrees
- moved Y1 0.89 mm to (86.0, 108.1)
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Connections:
- J1 pad 13: +3V3 -> Net-(J5-Pin_1)
- J1 pad 14: CMD -> Net-(J5-Pin_1)
- J1 pad 15: ~{PERST}/DAT3/CD -> Net-(J5-Pin_1)
- J1 pad 16: ~{CLKREQ}/DAT2 -> CMD
- J1 pad MP: (no net) -> GND
Routing:
- net DAT1: track 0.00 -> 99.3 mm, vias 0 -> 3
- net CMD: track 0.00 -> 98.2 mm, vias 0 -> 3
- net DAT0: track 0.00 -> 98.1 mm, vias 0 -> 3
- net CLK: track 0.00 -> 95.1 mm, vias 0 -> 3
- net DAT3/CD: track 5.15 -> 59.3 mm, vias 1 -> 3
- net DAT2: track 4.54 -> 57.9 mm, vias 1 -> 2
- net GND: track 0.00 -> 50.9 mm, vias 0 -> 31
- net +1V8: track 0.00 -> 48.2 mm, vias 0 -> 4
- net ~{CLKREQ}/DAT2: track 0.00 -> 40.5 mm, vias 0 -> 2
- net ~{PERST}/DAT3/CD: track 0.00 -> 40.1 mm, vias 0 -> 2
- net +3V3: track 0.00 -> 32.6 mm, vias 0 -> 12
- net Net-(J2-DEVSLP): track 34.5 -> 20.7 mm
- net Net-(J5-Pin_1): track 0.00 -> 13.3 mm
- net ~{LED1}: track 47.7 -> 58.4 mm
- net Net-(J2-VIO_1.8V): track 37.2 -> 26.6 mm
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- added copper zone on In2.Cu, net +3V3
- added copper zone on In3.Cu, net +3V3
- added copper zone on B.Cu, net GND
- added copper zone on F.Cu, net GND
- added copper zone on In1.Cu, net GND
- added copper zone on In4.Cu, net GND
Other:
- board size 98.3 x 40.6 mm -> 99.3 x 40.6 mm
