File: fpc-to-m2_m_socket/fpc-to-m2_m_socket.kicad_sch (KiCad schematic)
At the start: 20 parts, among them J2 Bus_M.2_Socket_M, J3 Conn_01x08_Pin, J4 Conn_01x16_Socket, J5 Micro_SD_Card, Y1 ASDMB-xxxMHz

Commit message: WIP
Parts:
- removed J4: Conn_01x16_Socket, symbol Connector:Conn_01x16_Socket
- removed J5: Micro_SD_Card, symbol Connector:Micro_SD_Card
- removed Y1: ASDMB-xxxMHz, Oscillator:Oscillator_SMD_Abracon_ASDMB-4Pin_2.5x2.0mm, symbol Oscillator:ASDMB-xxxMHz
- added C6: 15pF, Capacitor_SMD:C_0402_1005Metric, symbol Device:C
- added J1: ~, m1cha:FPC-SMD_P1.00-16P_LCS-SJ-H2.5, symbol m1cha:usdex-fpc-connector
- added J4: ~, m1cha:TF-SMD_503398-1892, symbol m1cha:Molex uSD connector 503398-1892
- added Y1: OK2EL89CJI-111YLC-32.768K, Oscillator:Oscillator_SMD_Abracon_ASDMB-4Pin_2.5x2.0mm, symbol m1cha:OK2EL89CJI-111YLC-32.768K
- C1, C2, C3, C5: footprint (none) -> Capacitor_SMD:C_0402_1005Metric
- C4: value 10uF -> 0.1uF; footprint (none) -> Capacitor_SMD:C_0402_1005Metric
- D1: footprint (none) -> LED_SMD:LED_0805_2012Metric
- J2: footprint (none) -> m1cha:CONN-SMD_APCI0146-P001A
- J3: value Conn_01x08_Pin -> ~; footprint (none) -> Connector_PinHeader_2.54mm:PinHeader_1x08_P2.54mm_Vertical; now not fitted
- R1, R2, R3, R4, R6, R7: footprint (none) -> Resistor_SMD:R_0402_1005Metric
- R5: footprint (none) -> Resistor_SMD:R_0402_1005Metric; now not fitted
- U2: footprint ProLib_pcs_2025-04-29-2:UQFN-16_L2.6-W1.8-P0.40-BL -> m1cha:tmux1574; symbol m1cha:TMUX1574RSVR -> m1cha:TMUX1574RSVR-UQFN
Connections:
- net +1V8: now also J1.8 (Pin_8)
- net CLK: now also J1.12 (Pin_12), J4.5 (CLK)
- net CMD: now also J1.14 (Pin_14), J4.3 (CMD)
- net DAT0: now also U1.4 (DA-), J4.7 (DAT0); no longer U1.5 (DA+)
- net DAT1: now also U1.5 (DA+), J4.8 (DAT1); no longer U1.4 (DA-)
- net DAT2: now also J4.1 (DAT2)
- net DAT3/CD: now also U2.12 (S4A), J4.2 (CD/DAT3); no longer U2.3 (S2A)
- net GND: now also C6.2, J1.1 (Pin_1), J1.11 (Pin_11), J1.4 (Pin_4), J1.7 (Pin_7), J4.11 (EH), J4.6 (VSS), Y1.2 (GND)
- net PCIe_RX+: now also J1.2 (Pin_2)
- net PCIe_RX-: now also J1.3 (Pin_3)
- net PCIe_TX+: now also J1.6 (Pin_6)
- net PCIe_TX-: now also J1.5 (Pin_5)
- net REFCLK+: now also U1.6 (DB-); no longer U1.7 (DB+)
- net REFCLK-: now also U1.7 (DB+); no longer U1.6 (DB-)
- net SUSCLK: now also C6.1, Y1.3 (Out)
- net ~{CLKREQ}/DAT2: now also J1.16 (Pin_16)
- net ~{PERST}: now also U2.11 (S4B); no longer U2.4 (S2B)
- net ~{PERST}/DAT3/CD: now also U2.10 (D4), J1.15 (Pin_15); no longer U2.5 (D2)
- net at R5.1, R6.2: now also Y1.1 (Tri-state)
- net at C4.1, R4.2, R5.2: now also Y1.4 (VDD)
- net +3.3V renamed +3V3
- net +3V3: now also J1.13 (Pin_13), J4.4 (VDD)
- net REFCLK+/DAT0 renamed DATx/REFCLK-
- net DATx/REFCLK-: now also J1.9 (Pin_9)
- net REFCLK-/DAT1 renamed DATx/REFCLK+
- net DATx/REFCLK+: now also J1.10 (Pin_10)
- no-connect marks 20 -> 22
Other:
- moved on the sheet: C1, R2

Commit message: WIP
Other:
- moved on the sheet: C2, C3
Changed lines of the file:
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@@
 	(symbol
 		(lib_id "Device:C")
-		(at 170.18 68.58 0)
+		(at 182.88 68.58 0)
 		(unit 1)
 		(exclude_from_sim no)
@@
 		(fields_autoplaced yes)
 		(property "Reference" "C2"
-			(at 173.99 67.3099 0)
+			(at 186.69 67.3099 0)
 			(effects
 				(font
@@
 		)
 		(property "Value" "1uF"
-			(at 173.99 69.8499 0)
+			(at 186.69 69.8499 0)
 			(effects
 				(font
@@
 		)
 		(property "Footprint" "Capacitor_SMD:C_0402_1005Metric"
-			(at 171.1452 72.39 0)
+			(at 183.8452 72.39 0)
 			(effects
 				(font
@@
 		)
 		(property "Datasheet" "~"
-			(at 170.18 68.58 0)
+			(at 182.88 68.58 0)
 			(effects
 				(font
@@
 		)
 		(property "Description" "Unpolarized capacitor"
-			(at 170.18 68.58 0)
+			(at 182.88 68.58 0)
 			(effects
 				(font
@@
 	(symbol
 		(lib_id "power:GND")
-		(at 180.34 72.39 0)
+		(at 170.18 72.39 0)
 		(unit 1)
 		(exclude_from_sim no)
@@
 		(fields_autoplaced yes)
 		(property "Reference" "#PWR023"
-			(at 180.34 78.74 0)
+			(at 170.18 78.74 0)
 			(effects
 				(font
@@
 		)
 		(property "Value" "GND"
-			(at 180.34 77.47 0)
+			(at 170.18 77.47 0)
 			(effects
 				(font
@@
 		)
 		(property "Footprint" ""
-			(at 180.34 72.39 0)
+			(at 170.18 72.39 0)
 			(effects
 				(font
@@
 		)
 		(property "Datasheet" ""
-			(at 180.34 72.39 0)
+			(at 170.18 72.39 0)
 			(effects
 				(font
@@
 		)
 		(property "Description" "Power symbol creates a global label with name \"GND\" , ground"
-			(at 180.34 72.39 0)
+			(at 170.18 72.39 0)
 			(effects
 				(font
@@
 	(symbol
 		(lib_id "power:+3V3")
-		(at 170.18 64.77 0)
+		(at 182.88 64.77 0)
 		(unit 1)
 		(exclude_from_sim no)
@@
 		(fields_autoplaced yes)
 		(property "Reference" "#PWR052"
-			(at 170.18 68.58 0)
+			(at 182.88 68.58 0)
 			(effects
 				(font
@@
 		)
 		(property "Value" "+3V3"
-			(at 170.18 59.69 0)
+			(at 182.88 59.69 0)
 			(effects
 				(font
@@
 		)
 		(property "Footprint" ""
-			(at 170.18 64.77 0)
+			(at 182.88 64.77 0)
 			(effects
 				(font
@@
 		)
 		(property "Datasheet" ""
-			(at 170.18 64.77 0)
+			(at 182.88 64.77 0)
 			(effects
 				(font
@@
 		)
 		(property "Description" "Power symbol creates a global label with name \"+3V3\""
-			(at 170.18 64.77 0)
+			(at 182.88 64.77 0)
 			(effects
 				(font
@@
 	(symbol
 		(lib_id "Device:C")
-		(at 180.34 68.58 0)
+		(at 170.18 68.58 0)
 		(unit 1)
 		(exclude_from_sim no)
@@
 		(fields_autoplaced yes)
 		(property "Reference" "C3"
-			(at 184.15 67.3099 0)
+			(at 173.99 67.3099 0)
 			(effects
 				(font
@@
 		)
 		(property "Value" "0.1uF"
-			(at 184.15 69.8499 0)
+			(at 173.99 69.8499 0)
 			(effects
 				(font
@@
 		)
 		(property "Footprint" "Capacitor_SMD:C_0402_1005Metric"
-			(at 181.3052 72.39 0)
+			(at 171.1452 72.39 0)
 			(effects
 				(font
@@
 		)
 		(property "Datasheet" "~"
-			(at 180.34 68.58 0)
+			(at 170.18 68.58 0)
 			(effects
 				(font
@@
 		)
 		(property "Description" "Unpolarized capacitor"
-			(at 180.34 68.58 0)
+			(at 170.18 68.58 0)
 			(effects
 				(font
@@
 	(symbol
 		(lib_id "power:GND")
-		(at 170.18 72.39 0)
+		(at 182.88 72.39 0)
 		(unit 1)
 		(exclude_from_sim no)
@@
 		(fields_autoplaced yes)
 		(property "Reference" "#PWR021"
-			(at 170.18 78.74 0)
+			(at 182.88 78.74 0)
 			(effects
 				(font
@@
 		)
 		(property "Value" "GND"
-			(at 170.18 77.47 0)
+			(at 182.88 77.47 0)
 			(effects
 				(font
@@
 		)
 		(property "Footprint" ""
-			(at 170.18 72.39 0)
+			(at 182.88 72.39 0)
 			(effects
 				(font
@@
 		)
 		(property "Datasheet" ""
-			(at 170.18 72.39 0)
+			(at 182.88 72.39 0)
 			(effects
 				(font
@@
 		)
 		(property "Description" "Power symbol creates a global label with name \"GND\" , ground"
-			(at 170.18 72.39 0)
+			(at 182.88 72.39 0)
 			(effects
 				(font
@@
 	(symbol
 		(lib_id "power:+3V3")
-		(at 180.34 64.77 0)
+		(at 170.18 64.77 0)
 		(unit 1)
 		(exclude_from_sim no)
@@
 		(fields_autoplaced yes)
 		(property "Reference" "#PWR053"
-			(at 180.34 68.58 0)
+			(at 170.18 68.58 0)
 			(effects
 				(font
@@
 		)
 		(property "Value" "+3V3"
-			(at 180.34 59.69 0)
+			(at 170.18 59.69 0)
 			(effects
 				(font
@@
 		)
 		(property "Footprint" ""
-			(at 180.34 64.77 0)
+			(at 170.18 64.77 0)
 			(effects
 				(font
@@
 		)
 		(property "Datasheet" ""
-			(at 180.34 64.77 0)
+			(at 170.18 64.77 0)
 			(effects
 				(font
@@
 		)
 		(property "Description" "Power symbol creates a global label with name \"+3V3\""
-			(at 180.34 64.77 0)
+			(at 170.18 64.77 0)
 			(effects
 				(font

Commit message: almost done
Parts:
- added J5: Conn_01x02_Pin, Connector_PinHeader_2.54mm:PinHeader_1x02_P2.54mm_Vertical, symbol Connector:Conn_01x02_Pin
- J1: footprint m1cha:FPC-SMD_P1.00-16P_LCS-SJ-H2.5 -> m1cha:FPC-SMD_18P-P1.00_JS_AFA07-S18XXX
- Y1: footprint Oscillator:Oscillator_SMD_Abracon_ASDMB-4Pin_2.5x2.0mm -> m1cha:OSC-SMD_4P-L3.2-W2.5-BL_TG-5006CE
Connections:
- net +3V3: now also J5.2 (Pin_2); no longer J1.13 (Pin_13)
- net CMD: now also J1.16 (CMD); no longer J1.14 (Pin_14)
- net GND: now also J1.MP, J2.MP
- net ~{CLKREQ}/DAT2: now also J1.18 (~{CLKREQ}/DAT2); no longer J1.16 (Pin_16)
- net ~{PERST}/DAT3/CD: now also J1.17 (~{PERST}/DAT3/CD); no longer J1.15 (Pin_15)
- new net: J1.13 (+3V3), J1.14 (+3V3), J1.15 (+3V3), J5.1 (Pin_1)
Other:
- moved on the sheet: C1, C2, C3, C5, J4, R1
